Commit message: xacro作成中-crankとasiの準備

File: tokuken_robot_description/urdf/hekken.xacro (robot description, xacro)
@@ -1,6 +1,6 @@
 <robot name="hexa_robot" xmlns:xacro="http://ros.org/wiki/xacro">
-    <xacro:macro name="crank_left" params="parent child xyz rpy">
+    <xacro:macro name="crank_left" params="parent child xyz">
         <joint name="${child}_joint" type="continuous">
-            <origin xyz="${xyz}" rpy="${rpy}"/>
+            <origin xyz="${xyz}" rpy="0 0 0"/>
             <parent link="${parent}"/>
             <child link="${child}_link"/>
@@ -18,7 +18,7 @@
         </link>
     </xacro:macro>
-    <xacro:macro name="crank_right" params="parent child xyz rpy">
+    <xacro:macro name="crank_right" params="parent child xyz">
         <joint name="${child}_joint" type="continuous">
-            <origin xyz="${xyz}" rpy="${rpy}"/>
+            <origin xyz="${xyz}" rpy="0 0 0"/>
             <parent link="${parent}"/>
             <child link="${child}_link"/>
@@ -81,3 +81,9 @@
         </visual>
     </link>
+    <xacro:crank_left parent="body_link" child="b_crank" xyz="-0.1623 0.1375 0.013"/>
+    <xacro:crank_left parent="body_link" child="c_crank" xyz="-0.1623 0.0475 0.013"/>
+    <xacro:crank_right parent="body_link" child="d_crank" xyz="-0.0777 0.0475 0.013"/>
+    <xacro:crank_right parent="body_link" child="a_crank" xyz="-0.0777 0.1375 0.013"/>
+    <!--TODO : xyz, rpy-->
+    <xacro:asi_left parent="b_crank_link" child="b_asi_1" xyz="-0.1773 0 0" rpy="0 0 0"/>
 </robot>

Commit message: pathのエラーを修正

File: tokuken_robot_description/urdf/hekken.xacro (robot description, xacro)
@@ -28,5 +28,5 @@
             <visual>
                 <geometry>
-                    <mesh filename="package://tokuken_robot_description/model/base/crank1_collide_ad_blen_low2.stl"/>
+                    <mesh filename="package://tokuken_robot_description/models/base/crank1_collide_ad_blen_low2.stl"/>
                 </geometry>
                 <material name="red"/>
@@ -44,5 +44,5 @@
             <visual>
                 <geometry>
-                    <mesh filename="package://tokuken_robot_description/model/base/asi_2_blen_low.stl"/>
+                    <mesh filename="package://tokuken_robot_description/models/base/asi_2_blen_low.stl"/>
                 </geometry>
                 <material name="green">
@@ -62,5 +62,5 @@
             <visual>
                 <geometry>
-                    <mesh filename="package://tokuken_robot_description/model/base/asi_1_blen_low.stl"/>
+                    <mesh filename="package://tokuken_robot_description/models/base/asi_1_blen_low.stl"/>
                 </geometry>
                 <material name="green"/>
@@ -77,5 +77,5 @@
         <visual name="body">
             <geometry>
-                <mesh filename="package://tokuken_robot_description/model/base/base_blen_low_3.stl"/>
+                <mesh filename="package://tokuken_robot_description/models/base/base_blen_low_3.stl"/>
             </geometry>
         </visual>

Commit message: asi_b_1だけ計算

File: tokuken_robot_description/urdf/hekken.xacro (robot description, xacro)
@@ -39,5 +39,5 @@
             <parent link="${parent}"/>
             <child link="${child}_link"/>
-            <axis xyz="0 0 1"/>
+            <axis xyz="1 0 0"/>
         </joint>
         <link name="${child}_link">
@@ -57,5 +57,5 @@
             <parent link="${parent}"/>
             <child link="${child}_link"/>
-            <axis xyz="0 0 1"/>
+            <axis xyz="1 0 0"/>
         </joint>
         <link name="${child}_link">
@@ -86,4 +86,4 @@
     <xacro:crank_right parent="body_link" child="a_crank" xyz="-0.0777 0.1375 0.013"/>
     <!--TODO : xyz, rpy-->
-    <xacro:asi_left parent="b_crank_link" child="b_asi_1" xyz="-0.1773 0 0" rpy="0 0 0"/>
+    <xacro:asi_left parent="b_crank_link" child="b_asi_1" xyz="-0.1773 ${0.1375+0.005*sin(radians(30))} ${0.013-0.005*cos(radians(30))}" rpy="0 0 0"/>
 </robot>

Commit message: 回転軸の調整

File: tokuken_robot_description/urdf/hekken.xacro (robot description, xacro)
@@ -5,5 +5,5 @@
             <parent link="${parent}"/>
             <child link="${child}_link"/>
-            <axis xyz="0 0 1"/>
+            <axis xyz="1 0 0"/>
         </joint>
         <link name="${child}_link">
@@ -23,5 +23,5 @@
             <parent link="${parent}"/>
             <child link="${child}_link"/>
-            <axis xyz="0 0 1"/>
+            <axis xyz="1 0 0"/>
         </joint>
         <link name="${child}_link">

Commit message: collision要素&アクチュエータ要素の追加

File: tokuken_robot_description/urdf/hekken.xacro (robot description, xacro)
@@ -7,4 +7,13 @@
             <axis xyz="1 0 0"/>
         </joint>
+        <transmission name="${child}_move" type="SimpleTransmission">
+            <type>transmission_interface/SimpleTransmission</type>
+            <actuator name="${child}_motor">
+                <mechanicalReduction>1</mechanicalReduction>
+            </actuator>
+            <joint name="${child}_joint">
+                <hardwareInterface>hardware_interface/VelocityJointInterface</hardwareInterface>
+            </joint>
+        </transmission>
         <link name="${child}_link">
             <visual>
@@ -16,5 +25,15 @@
                 </material>
             </visual>
+            <collision>
+                <geometry>
+                    <mesh filename="package://tokuken_robot_description/models/base/crank2_collide_ad_blen_low2.stl"/>
+                </geometry>
+            </collision>
         </link>
+        <gazebo reference="${child}_link">
+            <material>Gazebo/Red</material>
+            <mu1 value="1.0" />
+            <mu2 value="1.0" />
+        </gazebo>
     </xacro:macro>
     <xacro:macro name="crank_right" params="parent child xyz">
@@ -25,4 +44,13 @@
             <axis xyz="1 0 0"/>
         </joint>
+        <transmission name="${child}_move" type="SimpleTransmission">
+            <type>transmission_interface/SimpleTransmission</type>
+            <actuator name="${child}_motor">
+                <mechanicalReduction>1</mechanicalReduction>
+            </actuator>
+            <joint name="${child}_joint">
+                <hardwareInterface>hardware_interface/VelocityJointInterface</hardwareInterface>
+            </joint>
+        </transmission>
         <link name="${child}_link">
             <visual>
@@ -32,5 +60,15 @@
                 <material name="red"/>
             </visual>
+            <collision>
+                <geometry>
+                    <mesh filename="package://tokuken_robot_description/models/base/crank1_collide_ad_blen_low2.stl"/>
+                </geometry>
+            </collision>
         </link>
+        <gazebo reference="${child}_link">
+            <material>Gazebo/Red</material>
+            <mu1 value="1.0" />
+            <mu2 value="1.0" />
+        </gazebo>
     </xacro:macro>
     <xacro:macro name="asi_left" params="parent child xyz rpy">
@@ -50,5 +88,15 @@
                 </material>
             </visual>
+            <collision>
+                <geometry>
+                    <mesh filename="package://tokuken_robot_description/models/base/asi_2_blen_low.stl"/>
+                </geometry>
+            </collision>
         </link>
+        <gazebo reference="${child}_link">
+            <material>Gazebo/Green</material>
+            <mu1 value="1.0" />
+            <mu2 value="1.0" />
+        </gazebo>
     </xacro:macro>
     <xacro:macro name="asi_right" params="parent child xyz rpy">
@@ -66,5 +114,15 @@
                 <material name="green"/>
             </visual>
+            <collision>
+                <geometry>
+                    <mesh filename="package://tokuken_robot_description/models/base/asi_1_blen_low.stl"/>
+                </geometry>
+            </collision>
         </link>
+        <gazebo reference="${child}_link">
+            <material>Gazebo/Green</material>
+            <mu1 value="1.0" />
+            <mu2 value="1.0" />
+        </gazebo>
     </xacro:macro>
     <link name="base_link"/>
@@ -80,5 +138,15 @@
             </geometry>
         </visual>
+        <collision>
+            <geometry>
+                <mesh filename="package://tokuken_robot_description/models/base/base_blen_low_3.stl"/>
+            </geometry>
+        </collision>
     </link>
+    <gazebo reference="body_link">
+        <material>Gazebo/Blue</material>
+        <mu1 value="1.0" />
+        <mu2 value="1.0" />
+    </gazebo>
     <xacro:crank_left parent="body_link" child="b_crank" xyz="-0.1623 0.1375 0.013"/>
     <xacro:crank_left parent="body_link" child="c_crank" xyz="-0.1623 0.0475 0.013"/>

Commit message: spawn hekken in gazebo

File: tokuken_robot_description/urdf/hekken.xacro (robot description, xacro)
@@ -6,4 +6,6 @@
             <child link="${child}_link"/>
             <axis xyz="1 0 0"/>
+            <limit velocity="10.0" effort="0.2" />
+            <dynamics damping="0.1"/>
         </joint>
         <transmission name="${child}_move" type="SimpleTransmission">
@@ -30,4 +32,9 @@
                 </geometry>
             </collision>
+            <inertial>
+				<origin xyz="-0.037341 -0.000000002377 -0.002966" rpy="0 0 0"/>
+				<mass value="0.111155"/>
+				<inertia ixx="0.00001696" ixy="-0.000005133807" ixz="0.000000043631" iyy="0.00003475" iyz="-0.00002165" izz="0.00003573"/>
+			</inertial>
         </link>
         <gazebo reference="${child}_link">
@@ -35,4 +42,5 @@
             <mu1 value="1.0" />
             <mu2 value="1.0" />
+            <selfCollide>true</selfCollide>
         </gazebo>
     </xacro:macro>
@@ -43,4 +51,6 @@
             <child link="${child}_link"/>
             <axis xyz="1 0 0"/>
+            <limit velocity="10.0" effort="0.2" />
+            <dynamics damping="0.1"/>
         </joint>
         <transmission name="${child}_move" type="SimpleTransmission">
@@ -65,4 +75,9 @@
                 </geometry>
             </collision>
+            <inertial>
+				<origin xyz="0.037341 -0.000000002377 -0.002966" rpy="0 0 0"/>
+				<mass value="0.111155"/>
+				<inertia ixx="0.00001696" ixy="0.000005133807" ixz="-0.000000043631" iyy="0.00003475" iyz="0.00002165" izz="0.00003573"/>
+			</inertial>
         </link>
         <gazebo reference="${child}_link">
@@ -70,4 +85,5 @@
             <mu1 value="1.0" />
             <mu2 value="1.0" />
+            <selfCollide>true</selfCollide>
         </gazebo>
     </xacro:macro>
@@ -93,4 +109,9 @@
                 </geometry>
             </collision>
+            <inertial>
+				<origin xyz="-0.0045155 -0.00563879 -0.00377687" rpy="0 0 0"/>
+				<mass value="0.010706"/>
+				<inertia ixx="0.000005401807" ixy="0.000000000185" ixz="0.000000000496" iyy="0.000003139093" iyz="-0.00000098431" izz="0.000002411247"/>
+			</inertial>
         </link>
         <gazebo reference="${child}_link">
@@ -98,4 +119,5 @@
             <mu1 value="1.0" />
             <mu2 value="1.0" />
+            <selfCollide>true</selfCollide>
         </gazebo>
     </xacro:macro>
@@ -119,4 +141,9 @@
                 </geometry>
             </collision>
+            <inertial>
+				<origin xyz="0.0044845 -0.00563879 -0.00377687" rpy="0 0 0"/>
+				<mass value="0.010706"/>
+				<inertia ixx="0.000005401807" ixy="0.000000000185" ixz="0.000000000496" iyy="0.000003139093" iyz="-0.00000098431" izz="0.000002411247"/>
+			</inertial>
         </link>
         <gazebo reference="${child}_link">
@@ -124,4 +151,5 @@
             <mu1 value="1.0" />
             <mu2 value="1.0" />
+            <selfCollide>true</selfCollide>
         </gazebo>
     </xacro:macro>
@@ -143,4 +171,9 @@
             </geometry>
         </collision>
+        <inertial>
+            <origin xyz="-0.12003 0.0885733 0.024818" rpy="0 0 0"/>
+            <mass value="0.323853"/>
+			<inertia ixx="0.001101" ixy="-0.000000019489" ixz="-0.00000032811" iyy="0.001144" iyz="-0.00002903" izz="0.001950"/>
+		</inertial>
     </link>
     <gazebo reference="body_link">
@@ -148,4 +181,5 @@
         <mu1 value="1.0" />
         <mu2 value="1.0" />
+        <selfCollide>true</selfCollide>
     </gazebo>
     <xacro:crank_left parent="body_link" child="b_crank" xyz="-0.1623 0.1375 0.013"/>
@@ -165,3 +199,10 @@
     <xacro:asi_right parent="d_crank_link" child="d_asi_2" xyz="0.033 0.0 -0.005" rpy="${radians(-8)} 0 0"/>
     <xacro:asi_right parent="d_crank_link" child="d_asi_3" xyz="0.051 ${-0.005*sin(radians(30))} ${-0.005*cos(radians(30))}" rpy="${radians(-52)} 0 0"/>
+    <gazebo>
+        <plugin name="gazebo_ros_control" filename="libgazebo_ros_control.so">
+            <robotNamespace>/hekken</robotNamespace>
+            <robotSimType>gazebo_ros_control/DefaultRobotHWSim</robotSimType>
+            <legacyModeNS>true</legacyModeNS>
+        </plugin>
+    </gazebo>
 </robot>

Commit message: クランクのメッシュの変更適用

File: tokuken_robot_description/urdf/hekken.xacro (robot description, xacro)
@@ -21,5 +21,6 @@
             <visual>
                 <geometry>
-                    <mesh filename="package://tokuken_robot_description/models/base/crank2_collide_ad_blen_low2.stl"/>
+                    <mesh filename="package://tokuken_robot_description/models/base/crank2_ad.stl"/>
+                    <!--<mesh filename="package://tokuken_robot_description/models/base/crank2_collide_ad_blen_low2.stl"/>-->
                 </geometry>
                 <material name="red">
@@ -29,5 +30,6 @@
             <collision>
                 <geometry>
-                    <mesh filename="package://tokuken_robot_description/models/base/crank2_collide_ad_blen_low2.stl"/>
+                    <mesh filename="package://tokuken_robot_description/models/base/crank2_ad.stl"/>
+                    <!--<mesh filename="package://tokuken_robot_description/models/base/crank2_collide_ad_blen_low2.stl"/>-->
                 </geometry>
             </collision>
@@ -42,5 +44,5 @@
             <mu1 value="1.0" />
             <mu2 value="1.0" />
-            <selfCollide>true</selfCollide>
+            <!--<selfCollide>true</selfCollide>-->
         </gazebo>
     </xacro:macro>
@@ -66,5 +68,6 @@
             <visual>
                 <geometry>
-                    <mesh filename="package://tokuken_robot_description/models/base/crank1_collide_ad_blen_low2.stl"/>
+                    <mesh filename="package://tokuken_robot_description/models/base/crank1_ad.stl"/>
+                    <!--<mesh filename="package://tokuken_robot_description/models/base/crank1_collide_ad_blen_low2.stl"/>-->
                 </geometry>
                 <material name="red"/>
@@ -72,5 +75,6 @@
             <collision>
                 <geometry>
-                    <mesh filename="package://tokuken_robot_description/models/base/crank1_collide_ad_blen_low2.stl"/>
+                    <mesh filename="package://tokuken_robot_description/models/base/crank1_ad.stl"/>
+                    <!--<mesh filename="package://tokuken_robot_description/models/base/crank1_collide_ad_blen_low2.stl"/>-->
                 </geometry>
             </collision>
@@ -85,5 +89,5 @@
             <mu1 value="1.0" />
             <mu2 value="1.0" />
-            <selfCollide>true</selfCollide>
+            <!--<selfCollide>true</selfCollide>-->
         </gazebo>
     </xacro:macro>
@@ -158,5 +162,5 @@
         <parent link="base_link"/>
         <child link="body_link"/>
-        <origin xyz="0.0 0.0 0.0" rpy="0 0 0"/>
+        <origin xyz="0.0 0.0 0.05" rpy="0 0 0"/>
     </joint>
     <link name="body_link">

Commit message: ポリゴン数を減らした

File: tokuken_robot_description/urdf/hekken.xacro (robot description, xacro)
@@ -21,5 +21,5 @@
             <visual>
                 <geometry>
-                    <mesh filename="package://tokuken_robot_description/models/base/crank2_ad.stl"/>
+                    <mesh filename="package://tokuken_robot_description/models/base/crank2_lowp_ad_07.stl"/>
                     <!--<mesh filename="package://tokuken_robot_description/models/base/crank2_collide_ad_blen_low2.stl"/>-->
                 </geometry>
@@ -30,5 +30,5 @@
             <collision>
                 <geometry>
-                    <mesh filename="package://tokuken_robot_description/models/base/crank2_ad.stl"/>
+                    <mesh filename="package://tokuken_robot_description/models/base/crank2_lowp_ad_07.stl"/>
                     <!--<mesh filename="package://tokuken_robot_description/models/base/crank2_collide_ad_blen_low2.stl"/>-->
                 </geometry>
@@ -44,4 +44,6 @@
             <mu1 value="1.0" />
             <mu2 value="1.0" />
+            <gravity>true</gravity>
+            <minDepth>0.001</minDepth>
             <!--<selfCollide>true</selfCollide>-->
         </gazebo>
@@ -68,5 +70,5 @@
             <visual>
                 <geometry>
-                    <mesh filename="package://tokuken_robot_description/models/base/crank1_ad.stl"/>
+                    <mesh filename="package://tokuken_robot_description/models/base/crank1_lowp_ad_07.stl"/>
                     <!--<mesh filename="package://tokuken_robot_description/models/base/crank1_collide_ad_blen_low2.stl"/>-->
                 </geometry>
@@ -75,5 +77,5 @@
             <collision>
                 <geometry>
-                    <mesh filename="package://tokuken_robot_description/models/base/crank1_ad.stl"/>
+                    <mesh filename="package://tokuken_robot_description/models/base/crank1_lowp_ad_07.stl"/>
                     <!--<mesh filename="package://tokuken_robot_description/models/base/crank1_collide_ad_blen_low2.stl"/>-->
                 </geometry>
@@ -89,4 +91,6 @@
             <mu1 value="1.0" />
             <mu2 value="1.0" />
+            <gravity>true</gravity>
+            <minDepth>0.001</minDepth>
             <!--<selfCollide>true</selfCollide>-->
         </gazebo>
@@ -102,4 +106,5 @@
             <visual>
                 <geometry>
+                    <!--<mesh filename="package://tokuken_robot_description/models/base/asi_2_blen_low_3_ad.stl"/>-->
                     <mesh filename="package://tokuken_robot_description/models/base/asi_2_blen_low.stl"/>
                 </geometry>
@@ -110,4 +115,5 @@
             <collision>
                 <geometry>
+                    <!--<mesh filename="package://tokuken_robot_description/models/base/asi_2_blen_low_3_ad.stl"/>-->
                     <mesh filename="package://tokuken_robot_description/models/base/asi_2_blen_low.stl"/>
                 </geometry>
@@ -123,4 +129,5 @@
             <mu1 value="1.0" />
             <mu2 value="1.0" />
+            <gravity>true</gravity>
             <selfCollide>true</selfCollide>
         </gazebo>
@@ -136,4 +143,5 @@
             <visual>
                 <geometry>
+                    <!--<mesh filename="package://tokuken_robot_description/models/base/asi_1_blen_low_3_ad.stl"/>-->
                     <mesh filename="package://tokuken_robot_description/models/base/asi_1_blen_low.stl"/>
                 </geometry>
@@ -142,5 +150,6 @@
             <collision>
                 <geometry>
-                    <mesh filename="package://tokuken_robot_description/models/base/asi_1_blen_low.stl"/>
+                    <mesh filename="package://tokuken_robot_description/models/base/asi_1_blen_low_3_ad.stl"/>
+                    <!--<mesh filename="package://tokuken_robot_description/models/base/asi_1_blen_low.stl"/>-->
                 </geometry>
             </collision>
@@ -156,4 +165,5 @@
             <mu2 value="1.0" />
             <selfCollide>true</selfCollide>
+            <gravity>true</gravity>
         </gazebo>
     </xacro:macro>
@@ -185,8 +195,11 @@
         <mu1 value="1.0" />
         <mu2 value="1.0" />
+        <gravity>true</gravity>
         <selfCollide>true</selfCollide>
+        <minDepth>0.001</minDepth>
     </gazebo>
     <xacro:crank_left parent="body_link" child="b_crank" xyz="-0.1623 0.1375 0.013"/>
     <xacro:crank_left parent="body_link" child="c_crank" xyz="-0.1623 0.0475 0.013"/>
+    <!--
     <xacro:crank_right parent="body_link" child="d_crank" xyz="-0.0777 0.0475 0.013"/>
     <xacro:crank_right parent="body_link" child="a_crank" xyz="-0.0777 0.1375 0.013"/>
@@ -210,3 +223,4 @@
         </plugin>
     </gazebo>
+    -->
 </robot>
