Commit message: わかったかもしれない

File: tokuken_robot_description/urdf/hekken.xacro (robot description, xacro)
@@ -22,5 +22,4 @@
                 <geometry>
                     <mesh filename="package://tokuken_robot_description/models/base/crank2_lowp_ad_07.stl"/>
-                    <!--<mesh filename="package://tokuken_robot_description/models/base/crank2_collide_ad_blen_low2.stl"/>-->
                 </geometry>
                 <material name="red">
@@ -31,5 +30,4 @@
                 <geometry>
                     <mesh filename="package://tokuken_robot_description/models/base/crank2_lowp_ad_07.stl"/>
-                    <!--<mesh filename="package://tokuken_robot_description/models/base/crank2_collide_ad_blen_low2.stl"/>-->
                 </geometry>
             </collision>
@@ -46,5 +44,4 @@
             <gravity>true</gravity>
             <minDepth>0.001</minDepth>
-            <!--<selfCollide>true</selfCollide>-->
         </gazebo>
     </xacro:macro>
@@ -71,5 +68,4 @@
                 <geometry>
                     <mesh filename="package://tokuken_robot_description/models/base/crank1_lowp_ad_07.stl"/>
-                    <!--<mesh filename="package://tokuken_robot_description/models/base/crank1_collide_ad_blen_low2.stl"/>-->
                 </geometry>
                 <material name="red"/>
@@ -78,5 +74,4 @@
                 <geometry>
                     <mesh filename="package://tokuken_robot_description/models/base/crank1_lowp_ad_07.stl"/>
-                    <!--<mesh filename="package://tokuken_robot_description/models/base/crank1_collide_ad_blen_low2.stl"/>-->
                 </geometry>
             </collision>
@@ -93,5 +88,4 @@
             <gravity>true</gravity>
             <minDepth>0.001</minDepth>
-            <!--<selfCollide>true</selfCollide>-->
         </gazebo>
     </xacro:macro>
@@ -106,5 +100,4 @@
             <visual>
                 <geometry>
-                    <!--<mesh filename="package://tokuken_robot_description/models/base/asi_2_blen_low_3_ad.stl"/>-->
                     <mesh filename="package://tokuken_robot_description/models/base/asi_2_blen_low.stl"/>
                 </geometry>
@@ -115,5 +108,4 @@
             <collision>
                 <geometry>
-                    <!--<mesh filename="package://tokuken_robot_description/models/base/asi_2_blen_low_3_ad.stl"/>-->
                     <mesh filename="package://tokuken_robot_description/models/base/asi_2_blen_low.stl"/>
                 </geometry>
@@ -130,5 +122,4 @@
             <mu2 value="1.0" />
             <gravity>true</gravity>
-            <selfCollide>true</selfCollide>
         </gazebo>
     </xacro:macro>
@@ -143,5 +134,4 @@
             <visual>
                 <geometry>
-                    <!--<mesh filename="package://tokuken_robot_description/models/base/asi_1_blen_low_3_ad.stl"/>-->
                     <mesh filename="package://tokuken_robot_description/models/base/asi_1_blen_low.stl"/>
                 </geometry>
@@ -151,5 +141,4 @@
                 <geometry>
                     <mesh filename="package://tokuken_robot_description/models/base/asi_1_blen_low_3_ad.stl"/>
-                    <!--<mesh filename="package://tokuken_robot_description/models/base/asi_1_blen_low.stl"/>-->
                 </geometry>
             </collision>
@@ -164,5 +153,4 @@
             <mu1 value="1.0" />
             <mu2 value="1.0" />
-            <selfCollide>true</selfCollide>
             <gravity>true</gravity>
         </gazebo>
@@ -196,10 +184,8 @@
         <mu2 value="1.0" />
         <gravity>true</gravity>
-        <selfCollide>true</selfCollide>
         <minDepth>0.001</minDepth>
     </gazebo>
     <xacro:crank_left parent="body_link" child="b_crank" xyz="-0.1623 0.1375 0.013"/>
     <xacro:crank_left parent="body_link" child="c_crank" xyz="-0.1623 0.0475 0.013"/>
-    <!--
     <xacro:crank_right parent="body_link" child="d_crank" xyz="-0.0777 0.0475 0.013"/>
     <xacro:crank_right parent="body_link" child="a_crank" xyz="-0.0777 0.1375 0.013"/>
@@ -223,4 +209,3 @@
         </plugin>
     </gazebo>
-    -->
 </robot>

Commit message: revoluteにした

File: tokuken_robot_description/urdf/hekken.xacro (robot description, xacro)
@@ -91,9 +91,10 @@
     </xacro:macro>
     <xacro:macro name="asi_left" params="parent child xyz rpy">
-        <joint name="${child}_joint" type="continuous">
+        <joint name="${child}_joint" type="revolute">
             <origin xyz="${xyz}" rpy="${rpy}"/>
             <parent link="${parent}"/>
             <child link="${child}_link"/>
             <axis xyz="1 0 0"/>
+            <limit lower="${radians(-52)}" upper="${radians(38)}" effort="1.0" velocity="10.0"/>
         </joint>
         <link name="${child}_link">
@@ -125,9 +126,10 @@
     </xacro:macro>
     <xacro:macro name="asi_right" params="parent child xyz rpy">
-        <joint name="${child}_joint" type="continuous">
+        <joint name="${child}_joint" type="revolute">
             <origin xyz="${xyz}" rpy="${rpy}"/>
             <parent link="${parent}"/>
             <child link="${child}_link"/>
             <axis xyz="1 0 0"/>
+            <limit lower="${radians(-52)}" upper="${radians(38)}" effort="1.0" velocity="10.0"/>
         </joint>
         <link name="${child}_link">
